File: open_src/microcontroller.kicad_sch (KiCad schematic)
At the start: 11 parts, among them J1 AVR-JTAG-10, SW1 SW_DPST_x2, U1 MGM240PB32VNA3

Commit message: Added trace
Still not yet cross checked
Connections:
- net +3.3v: now also U1.15 (VDD)
- net GND: now also U1.1 (GND), U1.14 (GND), U1.23 (GND), U1.32 (GND), U1.34 (GND), U1.35 (GND), U1.36 (GND)
Changed lines of the file:
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@@
 (kicad_sch (version 20230121) (generator eeschema)
   (paper "A4")
+  (junction (at 110.49 153.035) (diameter 0) (color 0 0 0 0)
+  )
+  (junction (at 106.68 153.035) (diameter 0) (color 0 0 0 0)
+  )
   (junction (at 66.04 82.55) (diameter 0) (color 0 0 0 0)
   )
   (junction (at 66.04 80.01) (diameter 0) (color 0 0 0 0)
   )
+  (junction (at 118.11 153.035) (diameter 0) (color 0 0 0 0)
+  )
+  (junction (at 114.3 153.035) (diameter 0) (color 0 0 0 0)
+  )
+  (junction (at 108.585 153.035) (diameter 0) (color 0 0 0 0)
+  )
   (junction (at 226.695 127.635) (diameter 0) (color 0 0 0 0)
   )
+  (junction (at 102.87 153.035) (diameter 0) (color 0 0 0 0)
+  )
   (junction (at 204.47 127.635) (diameter 0) (color 0 0 0 0)
   )
@@
     (stroke (width 0) (type default))
   )
+  (wire (pts (xy 121.92 153.035) (xy 118.11 153.035))
+    (stroke (width 0) (type default))
+  )
   (wire (pts (xy 217.17 102.235) (xy 223.52 102.235))
     (stroke (width 0) (type default))
@@
     (stroke (width 0) (type default))
   )
+  (wire (pts (xy 99.06 153.035) (xy 102.87 153.035))
+    (stroke (width 0) (type default))
+  )
   (wire (pts (xy 230.505 68.58) (xy 230.505 71.12))
     (stroke (width 0) (type default))
@@
     (stroke (width 0) (type default))
   )
+  (wire (pts (xy 118.11 146.685) (xy 118.11 153.035))
+    (stroke (width 0) (type default))
+  )
+  (wire (pts (xy 201.295 127.635) (xy 204.47 127.635))
+    (stroke (width 0) (type default))
+  )
+  (wire (pts (xy 121.92 146.685) (xy 121.92 153.035))
+    (stroke (width 0) (type default))
+  )
   (wire (pts (xy 135.89 113.665) (xy 140.97 113.665))
     (stroke (width 0) (type default))
@@
     (stroke (width 0) (type default))
   )
+  (wire (pts (xy 102.87 146.685) (xy 102.87 153.035))
+    (stroke (width 0) (type default))
+  )
+  (wire (pts (xy 102.87 153.035) (xy 106.68 153.035))
+    (stroke (width 0) (type default))
+  )
+  (wire (pts (xy 99.06 146.685) (xy 99.06 153.035))
+    (stroke (width 0) (type default))
+  )
   (wire (pts (xy 227.33 127.635) (xy 226.695 127.635))
     (stroke (width 0) (type default))
@@
     (stroke (width 0) (type default))
   )
+  (wire (pts (xy 108.585 153.035) (xy 108.585 159.385))
+    (stroke (width 0) (type default))
+  )
   (wire (pts (xy 135.89 126.365) (xy 140.97 126.365))
     (stroke (width 0) (type default))
@@
     (stroke (width 0) (type default))
   )
+  (wire (pts (xy 110.49 153.035) (xy 108.585 153.035))
+    (stroke (width 0) (type default))
+  )
+  (wire (pts (xy 118.11 153.035) (xy 114.3 153.035))
+    (stroke (width 0) (type default))
+  )
   (wire (pts (xy 215.9 68.58) (xy 230.505 68.58))
     (stroke (width 0) (type default))
   )
+  (wire (pts (xy 110.49 146.685) (xy 110.49 153.035))
+    (stroke (width 0) (type default))
+  )
   (wire (pts (xy 66.04 82.55) (xy 66.04 85.09))
     (stroke (width 0) (type default))
@@
     (stroke (width 0) (type default))
   )
+  (wire (pts (xy 106.68 146.685) (xy 106.68 153.035))
+    (stroke (width 0) (type default))
+  )
   (wire (pts (xy 78.105 128.905) (xy 85.09 128.905))
     (stroke (width 0) (type default))
@@
     (stroke (width 0) (type default))
   )
+  (wire (pts (xy 106.68 153.035) (xy 108.585 153.035))
+    (stroke (width 0) (type default))
+  )
+  (wire (pts (xy 114.3 153.035) (xy 110.49 153.035))
+    (stroke (width 0) (type default))
+  )
   (wire (pts (xy 217.17 109.855) (xy 224.155 109.855))
     (stroke (width 0) (type default))
   )
+  (wire (pts (xy 135.89 137.795) (xy 140.97 137.795))
+    (stroke (width 0) (type default))
+  )
   (wire (pts (xy 66.04 80.01) (xy 66.04 73.025))
     (stroke (width 0) (type default))
@@
     (stroke (width 0) (type default))
   )
+  (wire (pts (xy 114.3 146.685) (xy 114.3 153.035))
+    (stroke (width 0) (type default))
+  )
   (global_label "PTI_FRAME" (shape input) (at 78.105 128.905 180) (fields_autoplaced)
     (effects (font (size 1.27 1.27)) (justify right))
@@
     )
   )
+  (global_label "GND" (shape input) (at 201.295 127.635 180) (fields_autoplaced)
+    (effects (font (size 1.27 1.27)) (justify right))
+    (property "Intersheetrefs" "${INTERSHEET_REFS}" (at 194.4393 127.635 0)
+      (effects (font (size 1.27 1.27)) (justify right) hide)
+    )
+  )
   (global_label "+3.3v" (shape input) (at 66.04 73.025 90) (fields_autoplaced)
     (effects (font (size 1.27 1.27)) (justify left))
@@
     )
   )
+  (global_label "GND" (shape input) (at 108.585 159.385 270) (fields_autoplaced)
+    (effects (font (size 1.27 1.27)) (justify right))
+    (property "Intersheetrefs" "${INTERSHEET_REFS}" (at 108.585 166.2407 90)
+      (effects (font (size 1.27 1.27)) (justify right) hide)
+    )
+  )
   (global_label "SW0" (shape input) (at 140.97 108.585 0) (fields_autoplaced)
     (effects (font (size 1.27 1.27)) (justify left))
@@
     (effects (font (size 1.27 1.27)) (justify left))
     (property "Intersheetrefs" "${INTERSHEET_REFS}" (at 146.4347 116.205 0)
+      (effects (font (size 1.27 1.27)) (justify left) hide)
+    )
+  )
+  (global_label "+3.3v" (shape input) (at 140.97 137.795 0) (fields_autoplaced)
+    (effects (font (size 1.27 1.27)) (justify left))
+    (property "Intersheetrefs" "${INTERSHEET_REFS}" (at 149.519 137.795 0)
       (effects (font (size 1.27 1.27)) (justify left) hide)
     )
@@
     (pin "20")
     (pin "33")
+    (pin "15")
+    (pin "1")
+    (pin "14")
+    (pin "32")
+    (pin "35")
+    (pin "36")
+    (pin "34")
+    (pin "23")
     (instances
       (project "open_src"
